File: panel/ethernet_led_controller_panel.kicad_pcb (KiCad board)
At the start: 2 copper layers, 75.1 x 75.1 mm, 0 parts

Commit message: updating any changes in hre ?
Other:
- board size 75.1 x 75.1 mm -> 75.1 x 85.1 mm
- board text added: "+V"
- board text added: "->"
- board text added: "5v <-> 12v"
- board text added: "CONTROLLER RESET"
- board text added: "D0"
- board text added: "D0-D3"
- board text added: "D4-D7"
- board text added: "LATERAL_LEDS v1_0_0 cyberboy666"
- board text added: "NETWORK CONNECTED"
- board text added: "POWER IN"
- board text added: "_^ 15"
- board text added: "lateral leds controller"
- board text added: "power input select"
- board text added: "power over serial"
- board text added: "underscores.shop"
- board text removed: "+5V"
- board text removed: "--"
- board text removed: "5V IN"
- board text removed: "CONNECT"
- board text removed: "D1-D4"
- board text removed: "D5-D8"
- board text removed: "D8"
- board text removed: "DTR"
- board text removed: "LINK"
- board text removed: "RTS"
- board text removed: "RX"
- board text removed: "TX"
- board text removed: "ethernet led controller"
